File: Hardware/KiCad/ThunderKillV2/ThunderKillV2.kicad_sch (KiCad schematic)
At the start: 0 parts

Commit message: Updated to fix 3d file paths, and updated page settings with version number and author.
Also updated the name for ThunderKILL V1
Other:
- company: (none) -> RoseDaggerDev                                               Original Credits: YveltalGriffin
- title: (none) -> ThunderKILL
Changed lines of the file:
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@@
 	(generator_version "9.0")
 	(paper "A4")
+	(title_block
+		(title "ThunderKILL")
+		(date "2025-09-05")
+		(rev "2.1")
+		(company "RoseDaggerDev                                               Original Credits: YveltalGriffin")
+	)
 	(polyline
 		(pts
