File: Hardware/KiCad/ThunderKillV2/ThunderKillV2.kicad_pcb (KiCad board)
At the start: 4 copper layers, 53.3 x 54.8 mm, 139 parts, among them IC1 EMC2103-2-AP-TR, IC2 BQ25622ERYKR, IC3 LS2406ERQ23, IC4 MAX20343BEWE+T, IC5 INA236AIYBJR, IC6 LP5810AYBHR, Q1 CSD23382F4, Q2 PNP, Q3 NX7002BKMYL, Q4 BC856BMBYL, Q5 BC856BMBYL, U1 TPS628682ARQYR, U2 TPS628681ARQYR, U3 TPS63810YFFR, U4 RT1715WSC, U5 PAC1934x-xJ6CX, U6 ATTINY1616-MNR, U7 LP5907UVX-1.8_NOPB, U8 TPS628681ARQYR

Commit message: Updating to newest local version
Parts:
- removed the G*** at (147.2, 104.4)
- added G***: LOGO, LOGO, F.Cu at (122.0, 75.2)
- added G***: LOGO, LOGO, F.Cu at (114.7, 90.7)
- added G***: LOGO, LOGO, F.Cu at (153.8, 103.9)
- added G***: LOGO, LOGO, F.Cu at (134.1, 114.7)
- added G***: LOGO, LOGO, F.Cu at (129.0, 98.5)
- added G***: LOGO, LOGO, B.Cu at (147.3, 104.4)
- added R24: 1k, Resistor_SMD:R_0402_1005Metric, F.Cu at (122.5, 101.3)
- added R25: 10k, Resistor_SMD:R_0402_1005Metric, F.Cu at (132.1, 104.3)
- added TP38: 1V0, RoseDaggerDev:TestPoint_Pad_3x1.0mm, B.Cu at (125.9, 97.6)
- added TP39: GND, RoseDaggerDev:TestPoint_Pad_3x1.0mm, B.Cu at (126.0, 106.8)
- added TP40: GND, RoseDaggerDev:TestPoint_Pad_3x1.0mm, B.Cu at (163.9, 92.3)
- added TP41: GND, RoseDaggerDev:TestPoint_Pad_3x1.0mm, B.Cu at (156.3, 125.5)
- added TP42: 1V15, RoseDaggerDev:TestPoint_Pad_3x1.0mm, B.Cu at (147.3, 125.6)
- C1, C10, C11, C12, C14, C15, C16, C18, C3, C40, C42, C43, C44, C46, C47, C48, C6, C7, C8, C9: value 22uF -> 22u
- C13, C17, C22, C28, C32, C4, C41, C45, C50: value 0.1uF -> 0.1u
- C2, C5: value 150uF -> 150u
- C23, C26: footprint Capacitor_SMD:C_0402_1005Metric -> Capacitor_SMD:C_0603_1608Metric
- C25: renamed from C49; value 0.1uF -> 0.1u
- C29, C34: value 1uF -> 1u
- C30: value 20u -> 22u; footprint Capacitor_SMD:C_0402_1005Metric -> Capacitor_SMD:C_0603_1608Metric
- C33, C39: footprint Capacitor_SMD:C_0603_1608Metric -> Capacitor_SMD:C_0402_1005Metric
- C37: value 1u -> 470n
- C38: footprint Capacitor_SMD:C_0805_2012Metric -> Capacitor_SMD:C_0603_1608Metric
- C49: renamed from C25; value 0.1uF -> 0.1u
- L1: footprint SamacSys_Parts:INDC3225X120N -> SamacSys_Parts:INDPM4442X150N
- L2, L6: footprint SamacSys_Parts:XFL5015152MEC -> SamacSys_Parts:INDPM4442X150N
- Q2: value PNP -> BC846; footprint SamacSys_Parts:SOT96P237X111-3N -> Package_TO_SOT_SMD:SOT-23
- Q5: value BC856BMBYL -> BC846
- TP22: footprint project-footprints:TestPoint_Pad_3x1.0mm -> RoseDaggerDev:TestPoint_Pad_3x1.0mm
- U5: value PAC1934x-xJ6CX -> PAC1934T-I/J6CX
- moved C8 3.21 mm to (128.3, 80.5)
- moved U1 3.21 mm to (128.1, 78.8)
- moved C1 2.97 mm to (120.8, 77.8), turned to -90 degrees
- moved R2 2.37 mm to (125.5, 78.7), turned to 180 degrees
- moved C3 2.32 mm to (119.6, 77.8), turned to -90 degrees
- moved C4 2.07 mm to (124.1, 78.2)
- moved C7 2.00 mm to (123.1, 77.8), turned to -90 degrees
- moved C24 1.68 mm to (135.8, 105.7)
- moved L1 1.32 mm to (126.7, 75.3)
- moved C6 1.10 mm to (121.9, 77.8), turned to -90 degrees
- moved R3 1.10 mm to (160.2, 84.5)
- moved C50 1.00 mm to (147.8, 122.4), turned to -90 degrees
- moved C9 0.98 mm to (160.7, 86.6), turned to 72 degrees
- moved R11 0.87 mm to (129.3, 103.7), turned to 90 degrees
- moved C20 0.85 mm to (133.0, 104.3)
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Connections:
- C25 pad 1: VDD -> GND
- C25 pad 2: GND -> VDD
- C45 pad 1: VDD -> +1V8
- C49 pad 1: GND -> +3V3
- C49 pad 2: VDD -> GND
- IC2 pad 3: unconnected-(IC2-~{PG}-Pad3) -> Net-(IC2-~{PG})
- IC4 pad B1: EN -> unconnected-(IC4-FAST-PadB1)
- IC5 pad B1: VDD -> +1V8
- IC5 pad D2: VDD -> +1V8
- IC6 pad B2: unconnected-(IC6-SYNC-PadB2) -> GND
- Q2 pad 2: Net-(IC1-DN2/DP3) -> Net-(IC1-DP2/DN3)
- Q2 pad 3: Net-(IC1-DP2/DN3) -> Net-(IC1-DN2/DP3)
- U4 pad B1: unconnected-(U4-VCONN-PadB1) -> Net-(U4-VCONN)
- U5 pad A1: +3V3 -> /Undervolt/3.3_OUT
- U5 pad A4: VDD -> +3V3
- U5 pad B1: /Undervolt/3.3_OUT -> +3V3
- U5 pad B3: unconnected-(U5-~{PWRDN}-PadB3) -> +1V8
- U5 pad C3: unconnected-(U5-SLOW-PadC3) -> GND
Routing:
- net VBUS: track 17.5 -> 28.8 mm
- net +3V3: track 51.2 -> 61.2 mm, vias 71 -> 44
- net PD_INT: track 51.9 -> 57.3 mm
- net EN: track 122.6 -> 127.8 mm, vias 6 -> 5
- net /Undervolt/1.0_OUT: track 25.6 -> 30.7 mm, vias 17 -> 10
- net +1V0: track 25.7 -> 30.3 mm, vias 32 -> 21
- net Net-(U1-VSET): track 4.25 -> 0.99 mm
- net SCL: track 131.8 -> 134.1 mm
- net +1V8: track 127.4 -> 129.7 mm, vias 54 -> 36
- net GND: track 2.83 -> 4.99 mm, vias 379 -> 242
- net /Undervolt/3.3_SW1: track 0.40 -> 2.25 mm, vias 8 -> 6
- net /Undervolt/3.3_SW2: track 0.40 -> 2.24 mm, vias 7 -> 6
- net /Undervolt/3.3_OUT: track 42.9 -> 44.6 mm
- net Net-(IC2-~{PG}): track 0.00 -> 1.48 mm
- net /Undervolt/1.15_OUT: track 23.9 -> 25.3 mm, vias 14 -> 9
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- added copper zone on B.Cu, net +1V0
- added copper zone on B.Cu, net +1V15
- added copper zone on B.Cu, net +1V8
- added copper zone on B.Cu, net +5V
- added copper zone on B.Cu, net /BMS/BAT_PORT_+
- added copper zone on B.Cu, net /BMS/BQ_SW
- added copper zone on B.Cu, net /BMS/PD_IN
- added copper zone on B.Cu, net /Undervolt/1.0_OUT
- added copper zone on B.Cu, net /Undervolt/1.0_SW
- added copper zone on B.Cu, net /Undervolt/1.15_OUT
- added copper zone on B.Cu, net /Undervolt/1.15_SW
- added copper zone on B.Cu, net /Undervolt/1.8_OUT
- added copper zone on B.Cu, net /Undervolt/1.8_SW
- added copper zone on B.Cu, net /Undervolt/3.3_SW1
- added copper zone on B.Cu, net /Undervolt/3.3_SW2
- added copper zone on B.Cu, net /Undervolt/5_SW1
- added copper zone on B.Cu, net /Undervolt/5_SW2
- added copper zone on B.Cu, net VDD
Other:
- board text added: "SDA SCL"
- board text added: "V${REVISION}"
- board text added: "Yvetal & Loopj 2024 _RoseDagger 2025"
- board text removed: "yveltal & loopj 2024 _Rosedagger 2025 V${REVISION}"
