File: Hardware/KiCad/ThunderKillV2/bms.kicad_sch (KiCad schematic)
At the start: 33 parts, among them IC2 BQ25622ERYKR, IC3 LS2406ERQ23, U4 RT1715WSC

Commit message: Updated to fix 3d file paths, and updated page settings with version number and author.
Also updated the name for ThunderKILL V1
Other:
- company: (none) -> RoseDaggerDev                                               Original Credits: YveltalGriffin
- title: (none) -> ThunderKILL
Changed lines of the file:
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@@
 	(generator_version "9.0")
 	(paper "A4")
+	(title_block
+		(title "ThunderKILL")
+		(date "2025-09-05")
+		(rev "2.1")
+		(company "RoseDaggerDev                                               Original Credits: YveltalGriffin")
+	)
 	(text "PD-BMS"
 		(exclude_from_sim no)

Commit message: Updating to newest local version
Parts:
- added R24: 1k, Resistor_SMD:R_0402_1005Metric, symbol Device:R_Small
- added R25: 10k, Resistor_SMD:R_0402_1005Metric, symbol Device:R
- C19, C27, C31: Digi-Key Part # (none) -> 490-14514-1-ND; Manufacturer_Name (none) -> Murata Electronics; Manufacturer_Part_Number (none) -> GCM155R71H104KE02J; Mouser Part Number (none) -> 81-GCM155R71H104KE2J
- C20: Digi-Key Part # (none) -> 490-GRM155C61E475ME15JCT-ND; Manufacturer_Name (none) -> Murata Electronics; Manufacturer_Part_Number (none) -> GRM155C61E475ME15J; Mouser Part Number (none) -> 81-GRM15C61E475ME15J
- C21: Digi-Key Part # (none) -> 490-10702-1-ND; Manufacturer_Name (none) -> Murata Electronics; Manufacturer_Part_Number (none) -> GRM155R71H473KE14D; Mouser Part Number (none) -> 81-GRM155R71H473KE4D
- C23, C26: footprint Capacitor_SMD:C_0402_1005Metric -> Capacitor_SMD:C_0603_1608Metric; Digi-Key Part # (none) -> 490-18214-1-ND; Manufacturer_Name (none) -> Murata Electronics; Manufacturer_Part_Number (none) -> GRM188R61E106KA73D; Mouser Part Number (none) -> 81-GRM188R61E106KA3D
- C24, C35: Digi-Key Part # (none) -> 490-10017-1-ND; Manufacturer_Name (none) -> Murata Electronics; Manufacturer_Part_Number (none) -> GRM155R61E105KA12D; Mouser Part Number (none) -> 81-GRM155R61E105KA2D
- C30: value 20u -> 22u; footprint Capacitor_SMD:C_0402_1005Metric -> Capacitor_SMD:C_0603_1608Metric; Digi-Key Part # (none) -> 490-GRM188C61E226ME01WCT-ND; Manufacturer_Name (none) -> Murata Electronics; Manufacturer_Part_Number (none) -> GRM188C61E226ME01W; Mouser Part Number (none) -> 81-GRM188C61E226ME1W
- C32: value 0.1uF -> 0.1u; Digi-Key Part # (none) -> 490-14514-1-ND; Manufacturer_Name (none) -> Murata Electronics; Manufacturer_Part_Number (none) -> GCM155R71H104KE02J; Mouser Part Number (none) -> 81-GCM155R71H104KE2J
- C33, C39: footprint Capacitor_SMD:C_0603_1608Metric -> Capacitor_SMD:C_0402_1005Metric; Digi-Key Part # (none) -> 490-GRM155C61E475ME15JCT-ND; Manufacturer_Name (none) -> Murata Electronics; Manufacturer_Part_Number (none) -> GRM155C61E475ME15J; Mouser Part Number (none) -> 81-GRM15C61E475ME15J
- C38: footprint Capacitor_SMD:C_0805_2012Metric -> Capacitor_SMD:C_0603_1608Metric; Digi-Key Part # (none) -> 490-18214-1-ND; Manufacturer_Name (none) -> Murata Electronics; Manufacturer_Part_Number (none) -> GRM188R61E106KA73D; Mouser Part Number (none) -> 81-GRM188R61E106KA3D
- F1: Digi-Key Part # (none) -> 18-0805L400SLWRCT-ND; MF (none) -> LITTELFUSE; MPN (none) -> 0805L400SLWR
- IC2: Digi-Key Part # (none) -> 296-BQ25622ERYKRCT-ND; MF (none) -> Texas Instruments
- IC3: Digi-Key Part # (none) -> 18-LS2406ERQ23CT-ND
- L4: Digi-Key Part # (none) -> 587-6422-1-ND
- R10: Digi-Key Part # (none) -> RMCF0402FT698RCT-ND; Manufacturer_Name (none) -> Stackpole Electronics Inc; Manufacturer_Part_Number (none) -> RMCF0402FT698R; Mouser Part Number (none) -> 708-RMCF0402FT698R
- R11: Digi-Key Part # (none) -> RMCF0402FT30K1CT-ND; Manufacturer_Name (none) -> Stackpole Electronics Inc; Manufacturer_Part_Number (none) -> RMCF0402FT30K1; Mouser Part Number (none) -> 708-RMCF0402FT30K1
- R15: Digi-Key Part # (none) -> RMCF0402FT3R60CT-ND; Manufacturer_Name (none) -> Stackpole Electronics Inc; Manufacturer_Part_Number (none) -> RMCF0402FT3R60; Mouser Part Number (none) -> 708-RMCF0402FT3R60
- R18: Digi-Key Part # (none) -> RMCF0402FT182KCT-ND; Manufacturer_Name (none) -> Stackpole Electronics Inc; Manufacturer_Part_Number (none) -> RMCF0402FT182K; Mouser Part Number (none) -> 708-RMCF0402FT182K
- R19: Digi-Key Part # (none) -> RMCF0402FT4K64CT-ND; Manufacturer_Name (none) -> Stackpole Electronics Inc; Manufacturer_Part_Number (none) -> RMCF0402FT4K64; Mouser Part Number (none) -> 708-RMCF0402FT4K64
- R20: Digi-Key Part # (none) -> 541-100KLCT-ND; Manufacturer_Name (none) -> Vishay Dale; Manufacturer_Part_Number (none) -> CRCW0402100KFKED; Mouser Part Number (none) -> 71-CRCW0402-100K-E3
- R9: Digi-Key Part # (none) -> RMCF0402FT5K23CT-ND; Manufacturer_Name (none) -> Stackpole Electronics Inc; Manufacturer_Part_Number (none) -> RMCF0402FT5K23; Mouser Part Number (none) -> 708-RMCF0402FT5K23
- TP11, TP15, TP17, TP20, TP22, TP26, TP27: now left out of the parts list
- U4: Digi-Key Part # (none) -> RT1715WSCCT-ND; Manufacturer_Name (none) -> Richtek; Manufacturer_Part_Number (none) -> RT1715WSC; Mouser Part Number (none) -> 835-RT1715WSC
Connections:
- net GND: now also R24.2
- net VDD: now also R25.1
- net at U4.B1 (VCONN): now also R24.1
- net at IC2.3 (~{PG}): now also R25.2
- no-connect marks 0 -> 2
