File: Hardware/KiCad/ThunderKillV2/mcu.kicad_sch (KiCad schematic)
At the start: 46 parts, among them IC1 EMC2103-2-AP-TR, IC6 LP5810AYBHR, Q1 CSD23382F4, Q2 PNP, Q3 NX7002BKMYL, Q4 BC856BMBYL, Q5 BC856BMBYL, U6 ATTINY1616-MNR, U7 LP5907UVX-1.8_NOPB

Commit message: Updated to fix 3d file paths, and updated page settings with version number and author.
Also updated the name for ThunderKILL V1
Other:
- company: (none) -> RoseDaggerDev                                               Original Credits: YveltalGriffin
- title: (none) -> ThunderKILL
Changed lines of the file:
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@@
 	(generator_version "9.0")
 	(paper "A4")
+	(title_block
+		(title "ThunderKILL")
+		(date "2025-09-05")
+		(rev "2.1")
+		(company "RoseDaggerDev                                               Original Credits: YveltalGriffin")
+	)

Commit message: Updating to newest local version
Parts:
- removed Q2: PNP, SamacSys_Parts:SOT96P237X111-3N, symbol Simulation_SPICE:PNP
- removed Q5: BC856BMBYL, SamacSys_Parts:BC856BMBYL, symbol SamacSys_Parts:BC856BMBYL
- added Q2: BC846, Package_TO_SOT_SMD:SOT-23, symbol Transistor_BJT:BC846
- added Q5: BC846, SamacSys_Parts:BC856BMBYL, symbol Transistor_BJT:BC846
- added TP39, TP40, TP41: GND, RoseDaggerDev:TestPoint_Pad_3x1.0mm, symbol Connector:TestPoint
- C2, C5: value 150uF -> 150u; Digi-Key Part # (none) -> 10-6TPS150MUDCT-ND; Manufacturer_Name (none) -> Panasonic Electronic Components; Manufacturer_Part_Number (none) -> 6TPS150MUD; Mouser Part Number (none) -> 667-6TPS150MUD
- C22, C25, C28: value 0.1uF -> 0.1u; Digi-Key Part # (none) -> 490-14514-1-ND; Manufacturer_Name (none) -> Murata Electronics; Manufacturer_Part_Number (none) -> GCM155R71H104KE02J; Mouser Part Number (none) -> 81-GCM155R71H104KE2J
- C29, C34: value 1uF -> 1u; Digi-Key Part # (none) -> 490-10017-1-ND; Manufacturer_Name (none) -> Murata Electronics; Manufacturer_Part_Number (none) -> GRM155R61E105KA12D; Mouser Part Number (none) -> 81-GRM155R61E105KA2D
- IC1: Digi-Key Part # (none) -> EMC2103-2-AP-CT-ND; MF (none) -> Microchip
- IC6: Digi-Key Part # (none) -> 296-LP5810AYBHRCT-ND
- Q1: Digi-Key Part # (none) -> 296-40003-1-ND
- Q3: Digi-Key Part # (none) -> 1727-2232-1-ND; Manufacturer_Name (none) -> Nexperia USA Inc.; Manufacturer_Part_Number (none) -> NX7002BKMYL; Mouser Part Number (none) -> 771-NX7002BKMYL
- Q4: Digi-Key Part # (none) -> 1727-2637-1-ND
- R13: Digi-Key Part # (none) -> RMCF0402FT133KCT-ND; Manufacturer_Name (none) -> Stackpole Electronics Inc; Manufacturer_Part_Number (none) -> RMCF0402FT133K; Mouser Part Number (none) -> 708-RMCF0402FT133K
- R14, R16, R17, R8: Digi-Key Part # (none) -> RMCF0402FT4K70CT-ND; Manufacturer_Name (none) -> Stackpole Electronics Inc; Manufacturer_Part_Number (none) -> RMCF0402FT4K70; Mouser Part Number (none) -> 708-RMCF0402FT4K70
- R6: Digi-Key Part # (none) -> RMCF0402FT49K9CT-ND; Manufacturer_Name (none) -> Stackpole Electronics Inc; Manufacturer_Part_Number (none) -> RMCF0402FT49K9; Mouser Part Number (none) -> 708-RMCF0402FT49K9
- R7: Digi-Key Part # (none) -> RMCF0402FT6K80; Manufacturer_Name (none) -> Stackpole Electronics Inc; Manufacturer_Part_Number (none) -> RMCF0402FT6K80; Mouser Part Number (none) -> 708-RMCF0402FT6K80
- TP10, TP12, TP13, TP14, TP16, TP18, TP19, TP21, TP23, TP24, TP28, TP29, TP30, TP31, TP32, TP34, TP36, TP37, TP4, TP7, TP8: now left out of the parts list
- U6: Digi-Key Part # (none) -> ATTINY1616-MNRCT-ND; Manufacturer_Name (none) -> Microchip Technology; Manufacturer_Part_Number (none) -> ATTINY1616-MNR; Mouser Part Number (none) -> 556-ATTINY1616MNR
- U7: Digi-Key Part # (none) -> 296-35634-1-ND
Connections:
- net GND: now also IC6.B2 (SYNC), TP39.1, TP40.1, TP41.1
- net at IC1.16 (DP2/DN3): now also Q2.2 (E), Q5.1 (B), Q5.3 (C)
- net at IC1.15 (DN2/DP3): now also Q2.1 (B), Q2.3 (C), Q5.2 (E)
