File: Hardware/KiCad/ThunderKillV2/undervolt.kicad_sch (KiCad schematic)
At the start: 59 parts, among them IC4 MAX20343BEWE+T, IC5 INA236AIYBJR, U1 TPS628682ARQYR, U2 TPS628681ARQYR, U3 TPS63810YFFR, U5 PAC1934x-xJ6CX, U8 TPS628681ARQYR

Commit message: Updated to fix 3d file paths, and updated page settings with version number and author.
Also updated the name for ThunderKILL V1
Other:
- company: (none) -> RoseDaggerDev                                               Original Credits: YveltalGriffin
- title: (none) -> ThunderKILL
Changed lines of the file:
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@@
 	(generator_version "9.0")
 	(paper "A4")
+	(title_block
+		(title "ThunderKILL")
+		(date "2025-09-05")
+		(rev "2.1")
+		(company "RoseDaggerDev                                               Original Credits: YveltalGriffin")
+	)
 	(text "1.8V DDR Buck"
 		(exclude_from_sim no)

Commit message: Updating to newest local version
Parts:
- added TP38: 1V0, RoseDaggerDev:TestPoint_Pad_3x1.0mm, symbol Connector:TestPoint
- added TP42: 1V15, RoseDaggerDev:TestPoint_Pad_3x1.0mm, symbol Connector:TestPoint
- C1, C10, C11, C12, C14, C15, C16, C18, C3, C40, C42, C43, C44, C46, C47, C48, C6, C7, C8, C9: value 22uF -> 22u; Digi-Key Part # (none) -> 490-GRM188C61E226ME01WCT-ND; Manufacturer_Name (none) -> Murata Electronics; Manufacturer_Part_Number (none) -> GRM188C61E226ME01W; Mouser Part Number (none) -> 81-GRM188C61E226ME1W
- C13, C17, C4, C41, C45, C49, C50: value 0.1uF -> 0.1u; Digi-Key Part # (none) -> 490-14514-1-ND; Manufacturer_Name (none) -> Murata Electronics; Manufacturer_Part_Number (none) -> GCM155R71H104KE02J; Mouser Part Number (none) -> 81-GCM155R71H104KE2J
- C36: Digi-Key Part # (none) -> 490-GRM188C61E226ME01WCT-ND; Manufacturer_Name (none) -> Murata Electronics; Manufacturer_Part_Number (none) -> GRM188C61E226ME01W; Mouser Part Number (none) -> 81-GRM188C61E226ME1W
- C37: value 1u -> 470n; Digi-Key Part # (none) -> 490-10017-1-ND; Manufacturer_Name (none) -> Murata Electronics; Manufacturer_Part_Number (none) -> GRM155R61E105KA12D; Mouser Part Number (none) -> 81-GRM155R61H474KE1D
- IC4: Digi-Key Part # (none) -> 175-MAX20343BEWE+TCT-ND
- IC5: Digi-Key Part # (none) -> 296-INA236AIYBJRCT-ND
- L1: footprint SamacSys_Parts:INDC3225X120N -> INDPM4442X150N; Digi-Key Part # (none) -> 283-MPI4015V2-R22-RCT-ND; Manufacturer_Name (none) -> Eaton; Manufacturer_Part_Number (none) -> MPI4015V2-R22-R; Mouser Part Number (none) -> 504-MPI4015V2-R22-R
- L2, L6: footprint SamacSys_Parts:XFL5015152MEC -> INDPM4442X150N; Digi-Key Part # (none) -> 283-MPI4015V2-R22-RCT-ND; Manufacturer_Name (none) -> Eaton; Manufacturer_Part_Number (none) -> MPI4015V2-R22-R; Mouser Part Number (none) -> 504-MPI4015V2-R22-R
- L3: Digi-Key Part # (none) -> 445-TFM201208BLE-R47MTCFCT-ND; Manufacturer_Name (none) -> TDK Corporation; Manufacturer_Part_Number (none) -> TFM201208BLE-R47MTCF; Mouser Part Number (none) -> 810-TFM201208BLER47M
- L5: Digi-Key Part # (none) -> 587-6422-1-ND
- R1, R21, R23, R3, R5: Digi-Key Part # (none) -> P19181CT-ND
- R12: Digi-Key Part # (none) -> RMCF0402FT3R60CT-ND; Manufacturer_Name (none) -> Stackpole Electronics Inc; Manufacturer_Part_Number (none) -> RMCF0402FT3R60; Mouser Part Number (none) -> 708-RMCF0402FT21K5
- R2: Digi-Key Part # (none) -> RMCF0402FT86K6CT-ND; Manufacturer_Name (none) -> Stackpole Electronics Inc; Manufacturer_Part_Number (none) -> RMCF0402FT86K6; Mouser Part Number (none) -> 708-RMCF0402FT86K6
- R22: Digi-Key Part # (none) -> 541-249KLCT-ND; Manufacturer_Name (none) -> Vishay Dale; Manufacturer_Part_Number (none) -> CRCW0402249KFKED; Mouser Part Number (none) -> 71-CRCW0402-249K-E3
- R4: Digi-Key Part # (none) -> RMCF0402FT133KCT-ND; Manufacturer_Name (none) -> Stackpole Electronics Inc; Manufacturer_Part_Number (none) -> RMCF0402FT133K; Mouser Part Number (none) -> 708-RMCF0402FT133K
- TP1, TP2, TP25, TP3, TP33, TP35, TP5, TP6, TP9: now left out of the parts list
- U1: Digi-Key Part # (none) -> 296-TPS628682ARQYRCT-ND; Manufacturer_Part_Number TPS628680ARQYR -> TPS628682ARQYR; Mouser Part Number 595-TPS628680ARQYR -> 595-TPS628682ARQYR
- U2, U8: Digi-Key Part # (none) -> 296-TPS628681ARQYRCT-ND; Manufacturer_Part_Number TPS628680ARQYR -> TPS628681ARQYR; Mouser Part Number 595-TPS628680ARQYR -> 595-TPS628681ARQYR
- U3: Digi-Key Part # (none) -> 296-TPS63810YFFRCT-ND
- U5: value PAC1934x-xJ6CX -> PAC1934T-I/J6CX; Digi-Key Part # (none) -> PAC1934T-I/J6CX-CT-ND; Manufacturer_Name (none) -> Microchip Technology; Manufacturer_Part_Number (none) -> PAC1934T-I/J6CX; Mouser Part Number (none) -> 579-PAC1934T-I/J6CX
Connections:
- net +1V0: now also TP38.1
- net +1V15: now also TP42.1
- net +1V8: now also C45.1, IC5.B1 (A0), IC5.D2 (VS), U5.B3 (~{PWRDN})
- net +3V3: now also C49.1, U5.A4 (V_{DD}), U5.B1 (SENSE2-); no longer U5.A1 (SENSE2+)
- net 3.3_OUT: now also U5.A1 (SENSE2+); no longer U5.B1 (SENSE2-)
- net EN: no longer IC4.B1 (FAST)
- net GND: now also U5.C3 (SLOW)
- net VDD: no longer C45.1, C49.1, IC5.B1 (A0), IC5.D2 (VS), U5.A4 (V_{DD})
- no-connect marks 0 -> 3
Other:
- moved on the sheet: TP25
